Commit message: update robot model (reduced box size)

File: robot_model/dual_panda_suhan.urdf.xacro (robot description, xacro)
@@ -10,5 +10,5 @@
       <origin xyz="0 0 0" rpy="0 0 0"/>
       <geometry>
-        <box size="1 2 1" />
+        <box size="0.3 0.9 1" />
       </geometry>
       <material name="White">
@@ -19,5 +19,5 @@
       <origin xyz="0 0 0" rpy="0 0 0"/>
       <geometry>
-        <box size="1 2 1" />
+        <box size="0.3 0.9 1" />
       </geometry>
     </collision>
